File: Schematics/ThetaProbe/ThetaProbe.kicad_pcb (KiCad board)
At the start: 2 copper layers, 83.8 x 52.1 mm, 13 parts, among them J1 BME280, J2 Relay_Module, J3 LED_Connection, J4 LED_Alive, J5 1-Wire CH1, J6 1-Wire CH2, J7 Power, U1 ESP32-DevKitC

Commit message: MeasurementPivot with tests done.
Parts:
- added R5: 4.7k, Resistor_THT:R_Axial_DIN0207_L6.3mm_D2.5mm_P7.62mm_Horizontal, F.Cu at (127.0, 68.6)
- added R6: 4.7k, Resistor_THT:R_Axial_DIN0207_L6.3mm_D2.5mm_P7.62mm_Horizontal, F.Cu at (127.0, 81.3)
Connections:
- U1 pad 11: unconnected-(U1-ADC2_CH7/GPIO27-Pad11) -> RELAY_1
- U1 pad 12: RELAY_1 -> unconnected-(U1-MTMS/GPIO14/ADC2_CH6-Pad12)
Routing:
- net +5V: track 87.4 -> 101.9 mm
- net +3V3: track 101.3 -> 114.0 mm
- net CH2_OneWire: track 19.4 -> 24.4 mm
- net GND: track 217.6 -> 222.5 mm
- net CH1_OneWire: track 23.0 -> 24.3 mm
- net RELAY_1: track 19.4 -> 20.1 mm
